Commit message: corrections in launch files and urdf

File: install/rubot_description/share/rubot_description/rover.urdf (robot description, URDF)
Before this commit: robot rover, 7 links, 6 joints
Links:
- added link base_footprint
Joints:
- added joint base_joint: type fixed, parent base_footprint, child chassis, origin xyz=0 0 0 rpy=0 0 0
